File: remote/remote.kicad_sch (KiCad schematic)
At the start: 6 parts, among them J1 Conn_01x10_Pin, SW1 SW_Push, SW2 SW_Push, U1 STM32L051C8Tx

Commit message: New versions
Parts:
- removed J1: Conn_01x10_Pin, Connector_FFC-FPC:Molex_200528-0100_1x10-1MP_P1.00mm_Horizontal, symbol Connector:Conn_01x10_Pin
- added Boot1, Reset1: TestPoint, TestPoint:TestPoint_Pad_2.0x2.0mm, symbol Connector:TestPoint
- added C1, C10, C2, C3, C4, C5, C7, C8, C9: 100n, Capacitor_SMD:C_0805_2012Metric_Pad1.18x1.45mm_HandSolder, symbol Device:C
- added C11, C6: 4.7u, Capacitor_SMD:C_0805_2012Metric_Pad1.18x1.45mm_HandSolder, symbol Device:C
- added D1, D2: LED, LED_SMD:LED_0805_2012Metric, symbol Device:LED
- added J1: Conn_01x08_Pin, Connector_PinHeader_2.54mm:PinHeader_2x04_P2.54mm_Vertical, symbol Connector:Conn_01x08_Pin
- added R1, R2: 100k, Resistor_SMD:R_0805_2012Metric, symbol Device:R
- added R3, R4: 10k, Resistor_SMD:R_0805_2012Metric, symbol Device:R
- renumbered SW2 to SW1, SW1 to SW2
Connections:
- net GND: now also BT1.2 (-), NRF1.2 (GND), SW1.2, SW2.2, U1.23 (VSS), U1.35 (VSS), U1.47 (VSS), U1.8 (VSSA), C1.2, C10.2, C11.2, C2.2, C3.2, C4.2, C5.2, C6.2, C7.2, C8.2, C9.1, J1.4 (Pin_4), R2.2
- net SWCLK: now also U1.37 (PA14), J1.1 (Pin_1)
- net SWDIO: now also U1.34 (PA13), J1.3 (Pin_3)
- net SW2: now reaches SW2.1
- net SW2: now also U1.46 (PB9), C10.1
- net +3V3: now reaches U1.1 (VDD)
- net +3V3: now also BT1.1 (+), NRF1.1 (VCC), U1.24 (VDD), U1.36 (VDDIO2), U1.48 (VDD), U1.9 (VDDA), C1.1, C11.1, C2.1, C3.1, C4.1, C5.1, C6.1, C7.1, D1.2 (A), D2.2 (A), J1.2 (Pin_2), R1.1
- net ADC_V_EXT: now reaches U1.10 (PA0)
- net LED_RED: now reaches U1.11 (PA1)
- net LED_RED: now also R3.2
- net LED_GREEN: now reaches U1.12 (PA2)
- net LED_GREEN: now also R4.2
- net SPI_SCK: now reaches U1.15 (PA5)
- net SPI_SCK: now also NRF1.5 (SCK)
- net SPI_MISO: now reaches U1.16 (PA6)
- net SPI_MISO: now also NRF1.7 (MISO)
- net SPI_MOSI: now reaches U1.17 (PA7)
- net SPI_MOSI: now also NRF1.6 (MOSI)
- net SPI_CSN: now reaches U1.18 (PB0)
- net SPI_CSN: now also NRF1.4 (CSN)
- net SPI_CE: now reaches U1.19 (PB1)
- net SPI_CE: now also NRF1.3 (CE)
- net SCL: now reaches U1.21 (PB10)
- net SCL: now also J1.6 (Pin_6)
- net SDA: now reaches U1.22 (PB11)
- net SDA: now also J1.8 (Pin_8)
- net USART1_TX: now reaches U1.30 (PA9)
- net USART1_TX: now also J1.7 (Pin_7)
- net USART1_RX: now reaches U1.31 (PA10)
- net USART1_RX: now also J1.5 (Pin_5)
- net SW1: now reaches U1.38 (PA15)
- net SW1: now also SW1.1, C9.2
- net BOOT: now reaches U1.44 (BOOT0)
- net BOOT: now also Boot1.1, R2.1
- net RESET: now reaches U1.7 (NRST)
- net RESET: now also C8.1, R1.2, Reset1.1
- new net: D2.1 (K), R4.1
- new net: D1.1 (K), R3.1
- no-connect marks 0 -> 17
Other:
- note added: "Boot/Reset"
- note added: "Buttons"
- note added: "Connectors"
- note added: "LEDs"
- note added: "NRF24"
- note added: "STM32L051"
- moved on the sheet: BT1, SW1, SW2
