File: ventilation/ventilation.kicad_sch (KiCad schematic)
At the start: 29 parts, among them J1 Conn_01x04_Pin, J2 Conn_01x04_Pin, J3 Conn_01x02_Pin, J4 Conn_01x03_Pin, Q2 IRLML6402, Q3 BC847, SW1 SW_Push, SW2 SW_Push, U1 STM32L051C8Tx

Commit message: Initial version
Parts:
- removed J1: Conn_01x04_Pin, Connector_Hirose:Hirose_DF13-04P-1.25DS_1x04_P1.25mm_Horizontal, symbol Connector:Conn_01x04_Pin
- removed J3: Conn_01x02_Pin, Connector_Hirose:Hirose_DF13-02P-1.25DS_1x02_P1.25mm_Horizontal, symbol Connector:Conn_01x02_Pin
- removed J4: Conn_01x03_Pin, Connector_Hirose:Hirose_DF13-03P-1.25DS_1x03_P1.25mm_Horizontal, symbol Connector:Conn_01x03_Pin
- removed SW1, SW2: SW_Push, PVDW_custom:SW_Push_4Pin, symbol PVDW_custom:SW_Push
- added C10, C11: 1u, Capacitor_SMD:C_0805_2012Metric_Pad1.18x1.45mm_HandSolder, symbol Device:C
- added J1: Conn_01x03_Pin, PVDW_custom:Connector_1x3_p2.54_hortizontal, symbol Connector:Conn_01x03_Pin
- added J3: Conn_01x04_Pin, PVDW_custom:Molex_PicoBlade_1x04_P1.25mm_Vertical, symbol Connector:Conn_01x04_Pin
- added J5: ~, PVDW_custom:Connector_1x2_p2.54_horizontal, symbol Connector:Conn_01x02_Pin
- added J7: Conn_01x02_Pin, PVDW_custom:Molex_PicoBlade_P1.25mm_Vertical, symbol Connector:Conn_01x02_Pin
- added R10, R9: 4k7, Resistor_SMD:R_0805_2012Metric_Pad1.20x1.40mm_HandSolder, symbol Device:R
- added R11: 470, Resistor_SMD:R_0805_2012Metric, symbol Device:R
- added U2: MCP1700x-330xxTT, Package_TO_SOT_SMD:SOT-23, symbol Regulator_Linear:MCP1700x-330xxTT
- C1, C2, C3: footprint (none) -> Capacitor_SMD:C_0805_2012Metric_Pad1.18x1.45mm_HandSolder
- C4: renamed from C8; footprint (none) -> Capacitor_SMD:C_0805_2012Metric_Pad1.18x1.45mm_HandSolder
- C5: renamed from C9; footprint (none) -> Capacitor_SMD:C_0805_2012Metric_Pad1.18x1.45mm_HandSolder
- C6: renamed from C4; footprint (none) -> Capacitor_SMD:C_0805_2012Metric
- C7: renamed from C5; footprint (none) -> Capacitor_SMD:C_0805_2012Metric_Pad1.18x1.45mm_HandSolder
- C8: renamed from C6; footprint (none) -> Capacitor_SMD:C_0805_2012Metric_Pad1.18x1.45mm_HandSolder
- C9: renamed from C10; footprint (none) -> Capacitor_SMD:C_0805_2012Metric
- D1, D2: footprint (none) -> LED_SMD:LED_0805_2012Metric
- J2: footprint Connector_Hirose:Hirose_DF13-04P-1.25DS_1x04_P1.25mm_Horizontal -> PVDW_custom:Molex_PicoBlade_53048-0410_1x04_P1.25mm_Horizontal
- R1, R2, R4, R5: footprint (none) -> Resistor_SMD:R_0805_2012Metric
- R3: renamed from R10; footprint (none) -> Resistor_SMD:R_0805_2012Metric_Pad1.20x1.40mm_HandSolder
- R6: renamed from R11; footprint (none) -> Resistor_SMD:R_0805_2012Metric_Pad1.20x1.40mm_HandSolder
- R7: renamed from R8; footprint (none) -> Resistor_SMD:R_0805_2012Metric
- R8: renamed from R9; footprint (none) -> Resistor_SMD:R_0805_2012Metric
- renumbered Q2 to Q1, Q3 to Q2
Connections:
- net +3V3: now also J2.2 (Pin_2), C11.1, R10.2, R9.1, U2.2 (VO); no longer J2.1 (Pin_1)
- net +BATT: now also Q1.2 (S), C10.1, J5.2 (Pin_2), U2.3 (VI); no longer Q1.3 (D)
- net BOOT: now also J7.1 (Pin_1)
- net GND: now also J2.1 (Pin_1), C10.2, C11.2, J1.1 (Pin_1), J5.1 (Pin_1), U2.1 (GND); no longer J2.2 (Pin_2)
- net I2C_SCL: now also R9.2
- net I2C_SDA: now also R10.1
- net LED_GREEN: now also U1.25 (PB12); no longer U1.21 (PB10)
- net LED_RED: now also U1.28 (PB15); no longer U1.22 (PB11)
- net RESET: now also J7.2 (Pin_2)
- net SIG_SERVO: now also J1.3 (Pin_3), R11.1; no longer U1.40 (PB4)
- net SWCLK: now also J3.1 (Pin_1)
- net SWDIO: now also J3.2 (Pin_2)
- net SW_SERVO: now also U1.6 (PH1); no longer U1.39 (PB3)
- net USART1_RX: now also J3.3 (Pin_3)
- net USART1_TX: now also J3.4 (Pin_4)
- net VCC_SERVO: now also Q1.3 (D), J1.2 (Pin_2); no longer Q1.2 (S)
- net B_NPN: now reaches Q2.1 (B), R6.2
- net G_FET: now reaches Q1.1 (G), Q2.3 (C), R3.1
- new net: R11.2, U1.39 (PB3)
Other:
- note added: "Power"
- note added: "STM32L051"
- note removed: "STM32L031"
- moved on the sheet: C6

Commit message: New version
Parts:
- added H1, H2: MountingHole, MountingHole:MountingHole_2.5mm, symbol Mechanical:MountingHole
Connections:
- net I2C_SCL: now also J2.3 (Pin_3); no longer J2.4 (Pin_4)
- net I2C_SDA: now also J2.4 (Pin_4); no longer J2.3 (Pin_3)
- net LED_GREEN: now also U1.28 (PB15); no longer U1.25 (PB12)
- net LED_RED: now also U1.25 (PB12); no longer U1.28 (PB15)
- net SIG_SERVO: now also J1.2 (Pin_2); no longer J1.3 (Pin_3)
- net SPI_CE: now also U1.22 (PB11); no longer U1.13 (PA3)
- net SPI_CSN: now also U1.21 (PB10); no longer U1.14 (PA4)
- net SW_SERVO: now also U1.12 (PA2); no longer U1.6 (PH1)
- net VCC_SERVO: now also J1.3 (Pin_3); no longer J1.2 (Pin_2)

Commit message: Changed SOT23 footprints to hand solder
Parts:
- Q1, Q2, U2: footprint Package_TO_SOT_SMD:SOT-23 -> Package_TO_SOT_SMD:TSOT-23_HandSoldering
Changed lines of the file:
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@@
 			)
 		)
-		(property "Footprint" "Package_TO_SOT_SMD:SOT-23"
+		(property "Footprint" "Package_TO_SOT_SMD:TSOT-23_HandSoldering"
 			(at 208.28 108.585 0)
 			(effects
@@
 			)
 		)
-		(property "Footprint" "Package_TO_SOT_SMD:SOT-23"
+		(property "Footprint" "Package_TO_SOT_SMD:TSOT-23_HandSoldering"
 			(at 44.45 155.575 0)
 			(effects
@@
 			)
 		)
-		(property "Footprint" "Package_TO_SOT_SMD:SOT-23"
+		(property "Footprint" "Package_TO_SOT_SMD:TSOT-23_HandSoldering"
 			(at 199.39 117.475 0)
 			(effects

Commit message: New version
Parts:
- added J4: Conn_01x04_Pin, PVDW_custom:Molex_PicoBlade_1x04_P1.25mm_Vertical, symbol Connector:Conn_01x04_Pin
Connections:
- net +3V3: now also J4.3 (Pin_3)
- net GND: now also J4.4 (Pin_4)
- net PA3: now reaches U1.13 (PA3)
- net PA3: now also J4.2 (Pin_2)
- net PA4: now reaches U1.14 (PA4)
- net PA4: now also J4.1 (Pin_1)
- no-connect marks 22 -> 20
Other:
- moved on the sheet: D1, D2, J5, R4, R5

Commit message: New version
Parts:
- removed C5: 100n, Capacitor_SMD:C_0805_2012Metric_Pad1.18x1.45mm_HandSolder, symbol Device:C
- removed J1: Conn_01x03_Pin, PVDW_custom:Connector_1x3_p2.54_hortizontal, symbol Connector:Conn_01x03_Pin
- removed J4: Conn_01x04_Pin, PVDW_custom:Molex_PicoBlade_1x04_P1.25mm_Vertical, symbol Connector:Conn_01x04_Pin
- removed J5: ~, PVDW_custom:Connector_1x2_p2.54_horizontal, symbol Connector:Conn_01x02_Pin
- removed J7: Conn_01x02_Pin, PVDW_custom:Molex_PicoBlade_P1.25mm_Vertical, symbol Connector:Conn_01x02_Pin
- added J6: Conn_01x10_Pin, PVDW_custom:FFC_1x10_P1.00mm_Horizontal, symbol Connector:Conn_01x10_Pin
- J2: footprint PVDW_custom:Molex_PicoBlade_53048-0410_1x04_P1.25mm_Horizontal -> PVDW_custom:Connector_1x4_p2.54_hortizontal
- J3: footprint PVDW_custom:Molex_PicoBlade_1x04_P1.25mm_Vertical -> PVDW_custom:Connector_1x4_p2.54_hortizontal
Connections:
- net PA3 is gone; now on net SW_SERVO: U1.13 (PA3)
- net +3V3: now also J6.2 (Pin_2)
- net +BATT: now also J3.2 (Pin_2)
- net BOOT: now also J6.9 (Pin_9)
- net GND: now also J3.1 (Pin_1), J6.1 (Pin_1)
- net I2C_SCL: now also U1.45 (PB8); no longer U1.42 (PB6)
- net I2C_SDA: now also U1.46 (PB9); no longer U1.43 (PB7)
- net LED_GREEN: now also U1.12 (PA2); no longer U1.28 (PB15)
- net LED_RED: now also U1.11 (PA1); no longer U1.25 (PB12)
- net RESET: now also J6.10 (Pin_10)
- net SIG_SERVO: now also J3.3 (Pin_3)
- net SWCLK: now also J6.8 (Pin_8); no longer J3.1 (Pin_1)
- net SWDIO: now also J6.7 (Pin_7); no longer J3.2 (Pin_2)
- net SW_SERVO: no longer U1.12 (PA2)
- net USART1_RX: now also J6.6 (Pin_6); no longer J3.3 (Pin_3)
- net USART1_TX: now also J6.5 (Pin_5); no longer J3.4 (Pin_4)
- net VCC_SERVO: now also J3.4 (Pin_4)
- net PB14: now reaches U1.27 (PB14)
- net PB14: now also J6.3 (Pin_3)
- net PA4: no longer names the net of U1.14 (PA4)
- new net PB15: J6.4 (Pin_4), U1.28 (PB15)
Other:
- moved on the sheet: R10, R9

Commit message: New versions
Parts:
- removed J6: Conn_01x10_Pin, PVDW_custom:FFC_1x10_P1.00mm_Horizontal, symbol Connector:Conn_01x10_Pin
- added J1: Conn_01x10_Pin, Connector_PinHeader_2.54mm:PinHeader_2x05_P2.54mm_Vertical, symbol Connector:Conn_01x10_Pin
- Q1, Q2, U2: footprint Package_TO_SOT_SMD:TSOT-23_HandSoldering -> Package_TO_SOT_SMD:SOT-23
Connections:
- net +3V3: now also J2.1 (Pin_1), J1.2 (Pin_2); no longer J2.2 (Pin_2)
- net BOOT: now also J1.10 (Pin_10)
- net GND: now also J2.2 (Pin_2), J1.1 (Pin_1); no longer J2.1 (Pin_1)
- net I2C_SCL: now also J2.4 (Pin_4); no longer J2.3 (Pin_3)
- net I2C_SDA: now also J2.3 (Pin_3); no longer J2.4 (Pin_4)
- net PB14: now also J1.4 (Pin_4)
- net PB15: now also J1.3 (Pin_3)
- net RESET: now also J1.9 (Pin_9)
- net SWCLK: now also J1.7 (Pin_7)
- net SWDIO: now also J1.8 (Pin_8)
- net USART1_RX: now also J1.5 (Pin_5)
- net USART1_TX: now also J1.6 (Pin_6)

Commit message: Order versions
Parts:
- removed J1: Conn_01x10_Pin, Connector_PinHeader_2.54mm:PinHeader_2x05_P2.54mm_Vertical, symbol Connector:Conn_01x10_Pin
- added Boot1, Reset1: TestPoint, TestPoint:TestPoint_Pad_2.0x2.0mm, symbol Connector:TestPoint
- added J4: Conn_01x08_Pin, Connector_PinHeader_2.54mm:PinHeader_2x04_P2.54mm_Vertical, symbol Connector:Conn_01x08_Pin
Connections:
- net +3V3: now also J4.2 (Pin_2)
- net BOOT: now also Boot1.1
- net GND: now also J4.4 (Pin_4)
- net PB14: now also J4.8 (Pin_8)
- net PB15: now also J4.6 (Pin_6)
- net RESET: now also Reset1.1
- net SWCLK: now also J4.1 (Pin_1)
- net SWDIO: now also J4.3 (Pin_3)
- net USART1_RX: now also J4.5 (Pin_5)
- net USART1_TX: now also J4.7 (Pin_7)
- net SIG_SERVO_OUT: now reaches R11.2, U1.39 (PB3)

Commit message: New order
Parts:
- removed Boot1, Reset1: TestPoint, TestPoint:TestPoint_Pad_2.0x2.0mm, symbol Connector:TestPoint
- removed J3: Conn_01x04_Pin, PVDW_custom:Connector_1x4_p2.54_hortizontal, symbol Connector:Conn_01x04_Pin
- added BOOT1, RESET1: SW_Push, PVDW_custom:SW_Push_4Pin, symbol PVDW_custom:SW_Push
- added C12: 10n, Capacitor_SMD:C_0805_2012Metric, symbol Device:C
- added J1: Conn_01x02_Pin, PVDW_custom:Connector_1x2_p2.54_horizontal, symbol Connector:Conn_01x02_Pin
- added J5: Conn_01x03_Pin, PVDW_custom:Connector_1x3_p2.54_hortizontal, symbol Connector:Conn_01x03_Pin
- added Q3: IRLML6402, Package_TO_SOT_SMD:SOT-23, symbol Transistor_FET:IRLML6402
- added R15: 0.1, Resistor_SMD:R_2512_6332Metric_Pad1.40x3.35mm_HandSolder, symbol Device:R
- added R16: 10k, Resistor_SMD:R_0805_2012Metric_Pad1.20x1.40mm_HandSolder, symbol Device:R
- added U3: INA180A1, Package_TO_SOT_SMD:SOT-23-5, symbol Amplifier_Current:INA180A1
- C6: value 100n -> 10n
- J4: footprint Connector_PinHeader_2.54mm:PinHeader_2x04_P2.54mm_Vertical -> Connector_PinHeader_2.54mm:PinHeader_1x08_P2.54mm_Vertical
- R1: value 100k -> 10k
- R3: value 40k -> 43k
- R4: value 10k -> 1k2
- R5: value 10k -> 820
- R6: value 40k -> 43k; footprint Resistor_SMD:R_0805_2012Metric_Pad1.20x1.40mm_HandSolder -> Resistor_SMD:R_0805_2012Metric
- R7: value 3k -> 3k3
- U2: footprint Package_TO_SOT_SMD:SOT-23 -> Package_TO_SOT_SMD:SOT-23_Handsoldering
Connections:
- net +3V3: now also J2.4 (Pin_4), BOOT1.1, Q3.2 (S), R16.1; no longer J2.1 (Pin_1)
- net +BATT: now also J1.2 (Pin_2)
- net BOOT: now also BOOT1.2
- net GND: now also J2.3 (Pin_3), J4.1 (Pin_1), C12.1, J1.1 (Pin_1), J5.1 (Pin_1), RESET1.1, U3.2 (GND); no longer J2.2 (Pin_2), J4.4 (Pin_4)
- net I2C_SCL: now also J2.1 (Pin_1); no longer J2.4 (Pin_4)
- net I2C_SDA: now also J2.2 (Pin_2); no longer J2.3 (Pin_3)
- net PB15: now also J4.7 (Pin_7); no longer J4.6 (Pin_6)
- net RESET: now also RESET1.2
- net SIG_SERVO: now also J5.2 (Pin_2)
- net SWCLK: now also J4.3 (Pin_3); no longer J4.1 (Pin_1)
- net SWDIO: now also J4.4 (Pin_4); no longer J4.3 (Pin_3)
- net SW_SERVO: now also U1.2 (PC13); no longer U1.13 (PA3)
- net USART1_TX: now also J4.6 (Pin_6); no longer J4.7 (Pin_7)
- net LED_GREEN_R: now reaches D2.1 (K), R5.1
- net LED_RED_R: now reaches D1.1 (K), R4.1
- net SW_I_SERVO: now reaches U1.14 (PA4)
- net SW_I_SERVO: now also Q3.1 (G), R16.2
- net VCC_SERVO renamed SHUNT_P
- net SHUNT_P: now also R15.2, U3.3 (+)
- new net INA_OUT: U1.13 (PA3), U3.1
- new net INA_VCC: C12.2, Q3.3 (D), U3.5 (V+)
- new net SHUNT_N: J5.3 (Pin_3), R15.1, U3.4 (-)
- no-connect marks 20 -> 18
Other:
- moved on the sheet: C6, C9, D1, D2, H1, H2, J2, J4, Q1, Q2, R1, R2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
