File: Sensor/Sensor/Sensor.kicad_pcb (KiCad board)
At the start: 2 copper layers, 20 x 50 mm, 42 parts, among them J31 Conn_Coaxial, J52 Conn_01x04_Pin, J53 Conn_01x06_Pin, U21 STM32L051C8Tx, U31 CC1101RGPR, Y31 26Mhz

Commit message: Added PCB for robot
Parts:
- added U51: SHTC3, PVDW_custom:shtc3, F.Cu at (107.7, 143.7)
- J52: footprint Connector_PinHeader_2.54mm:PinHeader_1x04_P2.54mm_Horizontal -> Connector_PinHeader_2.54mm:PinHeader_1x04_P2.54mm_Vertical
Routing:
- net /SDA: track 14.5 -> 22.2 mm
- net VCC: track 131.6 -> 136.5 mm, vias 7 -> 8
- net /SCL: track 11.5 -> 13.6 mm
- net GND: vias 68 -> 75
Other:
- board text added: "CLK"
- board text added: "DIO"
- board text added: "GND"
- board text added: "PVDW 2026 433MHZ"
- board text added: "PVDW 2026 STM32L051C8T6 CC1101 433MHZ SHTC03 (optional)"
- board text added: "RX"
- board text added: "SCL"
- board text added: "SDA"
- board text added: "TX"
- board text added: "VCC"
