File: Sensor/Sensor/Sensor.kicad_sch (KiCad schematic)
At the start: 42 parts, among them J31 Conn_Coaxial, J52 Conn_01x04_Pin, J53 Conn_01x06_Pin, U21 STM32L051C8Tx, U31 CC1101RGPR, Y31 26Mhz

Commit message: Added PCB for robot
Parts:
- added U51: SHTC3, PVDW_custom:shtc3, symbol PVDW_custom:SHTC3
- J52: footprint Connector_PinHeader_2.54mm:PinHeader_1x04_P2.54mm_Horizontal -> Connector_PinHeader_2.54mm:PinHeader_1x04_P2.54mm_Vertical
Connections:
- net GND: now also U51.4 (VSS), U51.5 (EXP)
- net SCL: now also U51.2 (SCL)
- net SDA: now also U51.3 (SDA)
- net VCC: now also U51.1 (VDD)
