File: Robot_remote/Robot_remote.kicad_pcb (KiCad board)
At the start: 2 copper layers, 85 x 100 mm, 16 parts, among them J1 Conn_01x05_Pin, J2 Conn_01x04_Pin, J3 Conn_01x12_Pin, U1 NRF24L01_Breakout, U2 CON**, U3 ESP32-S3-DEVKITC-1U-N8R8

Commit message: New versions for Robot PCBs
Routing:
- net /NRF_MOSI: track 93.1 -> 91.4 mm
- net /RY: track 14.7 -> 13.4 mm
- net /RX: track 14.7 -> 13.4 mm
- net /B2: track 14.8 -> 13.5 mm
- net /B1: track 14.8 -> 13.5 mm
- net /TRB: track 25.3 -> 24.1 mm
- net /TRA: track 25.3 -> 24.1 mm
- net /RES: track 25.3 -> 24.1 mm
- net /PUSH: track 25.3 -> 24.1 mm
- net /NRF_IRQ: track 45.8 -> 44.6 mm
- net /KEY0: track 25.3 -> 24.1 mm
- net /DC: track 25.3 -> 24.1 mm
- net /CS: track 25.3 -> 24.1 mm
- net /BLK: track 25.3 -> 24.1 mm
- net +5V: track 57.2 -> 58.5 mm
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